Commit message: Modified Robot URDF Model (Referance Frames changes), Cleaned up the Map Files.

File: install/butler_robot/share/butler_robot/model/robot.xacro (robot description, xacro)
@@ -52,11 +52,12 @@
 <!-- Include a file defining the Gazebo options and motion control driver-->
 <xacro:include filename="$(find butler_robot)/model/robot.gazebo"/>
-<!-- A dummy link and Joint-->
-<link name="base_footprint"/>
-  <joint name="base_joint" type="fixed">
-    <parent link="base_footprint"/>
-    <child link="body_link" />
-    <origin xyz="0 0 0.010" rpy="0 0 0"/>
-  </joint>
+<!-- Base Link-->
+<link name="base_link"/>
+<!-- Body Joint-->
+<joint name = "body_joint" type='fixed'>
+    <origin xyz = "${body_link_x_dim/2} 0 ${body_link_z_dim/2}" rpy='0 0 0'/>
+    <parent link = "base_link"/>
+    <child link = "body_link"/>
+</joint>
 <!-- Body Link-->
 <link name = 'body_link'>
@@ -84,8 +85,8 @@
 <!--Front Right Wheel-->
 <joint name = "front_wheel1_joint" type = "continuous">
-    <parent link = "body_link"/>
+    <parent link = "base_link"/>
     <child link = "front_wheel1_link"/>
-    <origin xyz = "${2*wheel_link_radius} ${-2*wheel_link_length} ${wheel_link_z_location}" rpy = "0 0 0"/>
-    <axis xyz = "0 1 0"/>
+    <origin xyz = "${body_link_x_dim} -${body_link_y_dim/2} 0" rpy = "${pi_const/2} 0 0"/>
+    <axis xyz = "0 0 -1"/>
     <limit effort = "1000" velocity = "1000"/>
     <dynamics damping = "1.0" friction = "1.0"/>
@@ -93,11 +94,9 @@
 <link name = "front_wheel1_link">
     <visual>
-        <origin rpy = "1.570795 0 0" xyz = "0 0 0"/>
-        <geometry>
-        <cylinder radius = "${wheel_link_radius}" length = "${wheel_link_length}"/>
-        </geometry>
-    </visual>
-    <collision>
-        <origin rpy = "1.570795 0 0" xyz = "0 0 0"/>
+        <geometry>
+        <cylinder radius = "${wheel_link_radius}" length = "${wheel_link_length}"/>
+        </geometry>
+    </visual>
+    <collision>
         <geometry>
         <cylinder radius = "${wheel_link_radius}" length = "${wheel_link_length}"/>
@@ -108,8 +107,8 @@
 <!--Rear Right Wheel-->
 <joint name = "rear_wheel1_joint" type = "continuous">
-    <parent link = "body_link"/>
+    <parent link = "base_link"/>
     <child link = "rear_wheel1_link"/>
-    <origin xyz = "${-2*wheel_link_radius} ${-2*wheel_link_length} ${wheel_link_z_location}" rpy = "0 0 0"/>
-    <axis xyz = "0 1 0"/>
+    <origin xyz = "0 -${body_link_y_dim/2} 0" rpy = "${pi_const/2} 0 0"/>
+    <axis xyz = "0 0 -1"/>
     <limit effort = "1000" velocity = "1000"/>
     <dynamics damping = "1.0" friction = "1.0"/>
@@ -117,11 +116,9 @@
 <link name = "rear_wheel1_link">
     <visual>
-        <origin rpy = "1.570795 0 0" xyz = "0 0 0"/>
-        <geometry>
-        <cylinder radius = "${wheel_link_radius}" length = "${wheel_link_length}"/>
-        </geometry>
-    </visual>
-    <collision>
-        <origin rpy = "1.570795 0 0" xyz = "0 0 0"/>
+        <geometry>
+        <cylinder radius = "${wheel_link_radius}" length = "${wheel_link_length}"/>
+        </geometry>
+    </visual>
+    <collision>
         <geometry>
         <cylinder radius = "${wheel_link_radius}" length = "${wheel_link_length}"/>
@@ -132,8 +129,8 @@
 <!--Front left Wheel-->
 <joint name = "front_wheel2_joint" type = "continuous">
-    <parent link = "body_link"/>
+    <parent link = "base_link"/>
     <child link = "front_wheel2_link"/>
-    <origin xyz = "${2*wheel_link_radius} ${2*wheel_link_length} ${wheel_link_z_location}" rpy = "0 0 0"/>
-    <axis xyz = "0 1 0"/>
+    <origin xyz = "${body_link_x_dim} ${body_link_y_dim/2} 0" rpy = "-${pi_const/2} 0 0"/>
+    <axis xyz = "0 0 1"/>
     <limit effort = "1000" velocity = "1000"/>
     <dynamics damping = "1.0" friction = "1.0"/>
@@ -141,11 +138,9 @@
 <link name = "front_wheel2_link">
     <visual>
-        <origin rpy = "1.570795 0 0" xyz = "0 0 0"/>
-        <geometry>
-        <cylinder radius = "${wheel_link_radius}" length = "${wheel_link_length}"/>
-        </geometry>
-    </visual>
-    <collision>
-        <origin rpy = "1.570795 0 0" xyz = "0 0 0"/>
+        <geometry>
+        <cylinder radius = "${wheel_link_radius}" length = "${wheel_link_length}"/>
+        </geometry>
+    </visual>
+    <collision>
         <geometry>
         <cylinder radius = "${wheel_link_radius}" length = "${wheel_link_length}"/>
@@ -156,8 +151,8 @@
 <!--Rear Left Wheel-->
 <joint name = "rear_wheel2_joint" type = "continuous">
-    <parent link = "body_link"/>
+    <parent link = "base_link"/>
     <child link = "rear_wheel2_link"/>
-    <origin xyz = "${-2*wheel_link_radius} ${2*wheel_link_length} ${wheel_link_z_location}" rpy = "0 0 0"/>
-    <axis xyz = "0 1 0"/>
+    <origin xyz = "0 ${body_link_y_dim/2} 0" rpy = "-${pi_const/2} 0 0"/>
+    <axis xyz = "0 0 1"/>
     <limit effort = "1000" velocity = "1000"/>
     <dynamics damping = "1.0" friction = "1.0"/>
@@ -165,11 +160,9 @@
 <link name = "rear_wheel2_link">
     <visual>
-        <origin rpy = "1.570795 0 0" xyz = "0 0 0"/>
-        <geometry>
-        <cylinder radius = "${wheel_link_radius}" length = "${wheel_link_length}"/>
-        </geometry>
-    </visual>
-    <collision>
-        <origin rpy = "1.570795 0 0" xyz = "0 0 0"/>
+        <geometry>
+        <cylinder radius = "${wheel_link_radius}" length = "${wheel_link_length}"/>
+        </geometry>
+    </visual>
+    <collision>
         <geometry>
         <cylinder radius = "${wheel_link_radius}" length = "${wheel_link_length}"/>
@@ -295,3 +288,55 @@
 </sensor>
 </gazebo>
+<!-- IMU Frame-->
+<joint name = "IMU_joint" type = "fixed">
+    <parent link = "head_link"/>
+    <child link = "IMU_frame"/>
+    <origin xyz = "0 ${head_link_radius} 0" rpy = "0 0 0"/>
+</joint>
+<link name = "IMU_frame">
+    <visual>
+        <origin rpy = "0 0 0" xyz = "0 0 0"/>
+        <geometry>
+        <sphere radius = "0.01"/>
+        </geometry>
+    </visual>
+    <collision>
+        <origin rpy = "0 0 0" xyz = "0 0 0"/>
+        <geometry>
+        <sphere radius = "0.01"/>
+        </geometry>
+    </collision>
+    <xacro:inertal_head/>
+</link>
+<!-- IMU Sensor -->
+<gazebo reference = 'IMU_frame'>
+ <sensor name="imu_sensor" type="imu">
+    <pose>0 0 0.1 0 0 0</pose>
+    <update_rate>100</update_rate>
+    <imu>
+      <angular_velocity>
+        <noise type="gaussian">
+          <mean>0</mean>
+          <stddev>0.02</stddev>
+        </noise>
+      </angular_velocity>
+      <linear_acceleration>
+        <noise type="gaussian">
+          <mean>0</mean>
+          <stddev>0.02</stddev>
+        </noise>
+      </linear_acceleration>
+    </imu>
+    <plugin name="imu_plugin" filename="libgazebo_ros_imu_sensor.so">
+        <frame_name>IMU_frame</frame_name>
+        <ros>
+          <namespace>/</namespace>
+          <remapping>imu/data_raw:=/imu/data</remapping>
+        </ros>
+        <update_rate>100</update_rate>
+        <bias_correction>true</bias_correction>
+        <gaussian_noise>0.001</gaussian_noise>
+      </plugin>
+  </sensor>
+</gazebo>
 </robot>
